File: Microhard_DB9_Supply.sch (EAGLE design)
At the start: 25 parts, among them IC1 FT232RL, IC2 SP213ECA-L, X1 PN61729-S, X2 D-SUB9-H2M09RA

Commit message: added Board and updated Schematics
Parts:
- added L3, L4, L5: Ferrite Bead, inductors:BLM15HB121SN1
- C10, C11: value 220uF -> 4.7uF; device adafruit:CPOL-USE10-20 -> rcl:CPOL-USD
- L1: SPICEPREFIX (none) -> L
Connections:
- net N$2: now also L3.1, L4.1, L5.1
- net VCC: now also L3.2, L4.2, L5.2
Other:
- moved on the sheet: C3
